File: Mir.sch (KiCad schematic (older format))
At the start: 45 parts, among them Q1 NSS40301MZ4T1G, SW1 SW_PUSH, U1 ATMEGA32U2-AU, Y1 16MHz

Commit message: Update to kicad5
Parts:
- C1, C2, C3, C4, C5, C6, CR1, CR10, CR11, CR12, CR13, CR14, CR2, CR3, CR4, CR5, CR6, CR7, CR8, CR9: symbol C_Small -> Device:C_Small
- F1: symbol Polyfuse_Small -> Device:Polyfuse_Small
- Q1: symbol BCP51 -> Mir-rescue:BCP51
- R1, R2, R3, R4, R5: symbol R_Small -> Device:R_Small
- RGB1, RGB10, RGB11, RGB12, RGB13, RGB14, RGB2, RGB3, RGB4, RGB5, RGB6, RGB7, RGB8, RGB9: symbol WS2812B -> Mir-rescue:WS2812B
- SW1: symbol SW_PUSH -> Mir-rescue:SW_PUSH
- U1: symbol ATMEGA32U2-AU -> Mir-rescue:ATMEGA32U2-AU
- USB1: symbol Molex-0548190589 -> Molex-0548190589:Molex-0548190589
- Y1: symbol Crystal_GND24_Small -> Device:Crystal_GND24_Small
