File: Mir.sch (KiCad schematic (older format))
At the start: 45 parts, among them Q1 NSS40301MZ4T1G, SW1 SW_PUSH, U1 ATMEGA32U2-AU, Y1 16MHz

Commit message: Route without MCU connections
Parts:
- removed CR10, CR11, CR12, CR13, CR14, CR9: 0.1u, Capacitors_SMD:C_0805_HandSoldering, symbol Device:C_Small
- removed Q1: NSS40301MZ4T1G, TO_SOT_Packages_SMD:SOT-223-3_TabPin2, symbol Mir-rescue:BCP51
- removed RGB10, RGB11, RGB12, RGB13, RGB14, RGB9: WS2812B, WS2812B:WS2812B, symbol Mir-rescue:WS2812B
- removed USB1: Molex-0548190589, Molex-0548190589:Molex-0548190589, symbol Molex-0548190589:Molex-0548190589
- added R6: 5.1k, Resistors_SMD:R_0603, symbol Device:R_Small
- added U2: PRTR5V0U2X, locallib:SOT143B, symbol ai03-locallib:PRTR5V0U2X
- added USB1: HRO-TYPE-C-31-M-12, Type-C:HRO-TYPE-C-31-M-12-Assembly, symbol Type-C:HRO-TYPE-C-31-M-12
- C1, C2, C3, C4, C5, C6, CR1, CR2, CR3, CR4, CR5, CR6, CR7, CR8: footprint Capacitors_SMD:C_0805_HandSoldering -> Capacitors_SMD:C_0603
- F1: footprint Fuse_Holders_and_Fuses:Fuse_SMD1206_HandSoldering -> Fuse_Holders_and_Fuses:Fuse_SMD1206_Reflow
- R1, R2, R3, R5: footprint Resistors_SMD:R_0805_HandSoldering -> Resistors_SMD:R_0603
- R4: value 1.5k -> 5.1k; footprint Resistors_SMD:R_0805_HandSoldering -> Resistors_SMD:R_0603
- SW1: footprint Molex-0548190589:PushButton_6x6mm_TH -> Molex-0548190589:SKQG-1155865
- U1: footprint Housings_QFP:TQFP-32_7x7mm_Pitch0.8mm -> Housings_DFN_QFN:QFN-32-1EP_5x5mm_Pitch0.5mm
- Y1: footprint Crystals:Crystal_SMD_3225-4pin_3.2x2.5mm_HandSoldering -> Crystals:Crystal_SMD_3225-4pin_3.2x2.5mm
Connections:
- net labels added: D+, D-
- net labels removed: COL0, COL1, COL2, COL3, COL4, COL5, COL6, COL7, DM, DP, D_N, D_P, LEDGND, ROW0, ROW1, ROW2, ROW3, ROW4, ROW5, ROW6, ROW7, ROW8, ROW9
- wire segments 177 -> 146
- no-connect marks 2 -> 3
Other:
- note added: "2018-11-28"
- note added: "Mir Keyboard\n"
- note removed: "2017-10-15\n"
- note removed: "This is supposed to be a NPN transistor\nFor some reason KiCad keeps flipping the arrow the other way"
- note removed: "Voyager Keyboard\n"
- moved on the sheet: F1, R2, R3

Commit message: Finish routing
Connections:
- net labels added: COL0, COL1, COL10, COL11, COL2, COL3, COL4, COL5, COL6, COL7, COL8, COL9, ROW0, ROW1, ROW2, ROW3
Changed lines of the file:
@@
 $EndComp
 Connection ~ 2100 6700
+Text GLabel 4250 3800 2    50   Input ~ 0
+COL0
+Text GLabel 4250 3900 2    50   Input ~ 0
+COL1
+Text GLabel 4250 2600 2    50   Input ~ 0
+COL2
+Text GLabel 4250 2500 2    50   Input ~ 0
+COL3
+Text GLabel 4250 2400 2    50   Input ~ 0
+COL4
+Text GLabel 4250 2300 2    50   Input ~ 0
+COL5
+Text GLabel 4250 2200 2    50   Input ~ 0
+COL6
+Text GLabel 4250 2100 2    50   Input ~ 0
+COL7
+Text GLabel 4250 2000 2    50   Input ~ 0
+COL8
+Text GLabel 4250 1900 2    50   Input ~ 0
+COL9
+Text GLabel 4250 3400 2    50   Input ~ 0
+COL10
+Text GLabel 4250 3300 2    50   Input ~ 0
+COL11
+Text GLabel 4250 3200 2    50   Input ~ 0
+ROW3
+Text GLabel 4250 3100 2    50   Input ~ 0
+ROW2
+Text GLabel 4250 3000 2    50   Input ~ 0
+ROW1
+Text GLabel 4250 2900 2    50   Input ~ 0
+ROW0
 $EndSCHEMATC

Commit message: Decorations
Changed lines of the file:
@@
 Text GLabel 4250 2900 2    50   Input ~ 0
 ROW0
+Text GLabel 4250 4000 2    50   Input ~ 0
+RGBLED
 $EndSCHEMATC
