File: Mir.kicad_pcb (KiCad board)
At the start: 2 copper layers, 285 x 94.6 mm, 258 parts, among them Q1 NSS40301MZ4T1G, SW1 SW_PUSH, U1 ATMEGA32U2-AU, Y1 16MHz

Commit message: Route without MCU connections
Parts:
- removed CR10, CR11, CR12, CR13, CR14, CR9: 0.1u, Capacitors_SMD:C_0805_HandSoldering
- removed D_#0_1, D_#1, D_#2, D_#3, D_#4, D_#5, D_#6, D_#7, D_#8, D_#9, D_'1, D_,1, D_-1, D_.1, D_/1, D_;1, D_=1, D_A1, D_ALT1, D_B1, D_BACK1, D_C1, D_CAPS1, D_CTRL1, D_D1, D_DEL1, D_DOWN1, D_E1, D_ENTER1, D_ESC1, D_F1, D_FN1, D_G1, D_H1, D_I1, D_ISO\1, D_ISO`1, D_J1, D_K1, D_L1, D_LEFT1, D_M1, D_N1, D_O1, D_P1, D_Q1, D_R1, D_RIGHT1, D_RSHIFT1, D_S1, D_SHIFT1, D_SPACE1, D_T1, D_TAB1, D_U1, D_UP1, D_V1, D_W1, D_WIN1, D_X1, D_Y1, D_Z1, D_[1, D_\1, D_]1, D_`1: SMA-GENERIC, Diodes_SMD:D_SOD-323_HandSoldering
- removed K_#0_1, K_#1, K_#2, K_#3, K_#4, K_#5, K_#6, K_#7, K_#8, K_#9, K_'1, K_,1, K_-1, K_.1, K_/2, K_;1, K_=1, K_A1, K_B1, K_BACK1, K_C1, K_D1, K_DEL1, K_DOWN1, K_E1, K_ESC1, K_F1, K_FN1, K_G1, K_H1, K_I1, K_ISO\1, K_ISO`1, K_J1, K_K1, K_L1, K_LEFT1, K_M1, K_N1, K_O1, K_P1, K_Q1, K_R1, K_RIGHT1, K_RSHIFT1, K_S1, K_T1, K_U1, K_UP1, K_V1, K_W1, K_X1, K_Y1, K_Z1, K_[1, K_]1, K_`1: MX-1U, MX_Alps_Hybrid:MX-1U
- removed K_/1, K_CAPS1: MX-1.75U, MX_Alps_Hybrid:MX-1.75U
- removed K_ALT1, K_CTRL1, K_RALT1, K_SHIFT2, K_WIN1: MX-1.25U, MX_Alps_Hybrid:MX-1.25U
- removed K_ALT2, K_CAPS2: MX-1.25U, MX_Alps_Hybrid:MX-1.25U-FLIPPED
- removed K_BACK2: MX-2U, MX_Alps_Hybrid:MX-2U
- removed K_CMD1, K_TAB1, K_\1: MX-1.5U, MX_Alps_Hybrid:MX-1.5U
- removed K_CTRL2, K_RCTRL2: MX-1.5U, MX_Alps_Hybrid:MX-1.5U-FLIPPED
- removed K_ENTER1, K_SHIFT1: MX-2.25U, MX_Alps_Hybrid:MX-2.25U
- removed K_ISOENTER1: MX-ISO, MX_Alps_Hybrid:MX-ISO-Combined-ReversedStabilizers
- removed K_RSHIFT2: MX-2.75U, MX_Alps_Hybrid:MX-2.75U-FLIPPED
- removed K_SPACE1: MX-6.25U-FLIPPED, MX_Alps_Hybrid:MX-6.25U-ReversedStabilizers
- removed K_SPACE2: MX-6.5U, MX_Alps_Hybrid:MX-6.5U
- removed Q1: NSS40301MZ4T1G, TO_SOT_Packages_SMD:SOT-223-3_TabPin2
- removed REF**: 60_Outline, local_lib:60_Outline
- removed REF** (x2): AI03-30Mil, ai03-logo:AI03-30Mil
- removed RGB10, RGB11, RGB12, RGB13, RGB14, RGB9: WS2812B, WS2812B:WS2812B
- removed R_#0_1, R_#1, R_#2, R_#3, R_#4, R_#5, R_#6, R_#7, R_#8, R_#9, R_'1, R_,1, R_-1, R_.1, R_/1, R_;1, R_=1, R_A1, R_ALT1, R_B1, R_BACK1, R_C1, R_CAPS1, R_CTRL1, R_D1, R_DEL1, R_DOWN1, R_E1, R_ENTER1, R_ESC1, R_F1, R_FN1, R_G1, R_H1, R_I1, R_ISO\1, R_ISO`1, R_J1, R_K1, R_L1, R_LEFT1, R_M1, R_N1, R_O1, R_P1, R_Q1, R_R1, R_RIGHT1, R_RSHIFT1, R_S1, R_SHIFT1, R_SPACE1, R_T1, R_TAB1, R_U1, R_UP1, R_V1, R_W1, R_WIN1, R_X1, R_Y1, R_Z1, R_[1, R_\1, R_]1, R_`1: 2.7k, Resistors_SMD:R_0805_HandSoldering
- added D1: SOD-123, Diodes_SMD:D_SOD-123, B.Cu at (49.2, 41.3)
- added D10: SOD-123, Diodes_SMD:D_SOD-123, B.Cu at (220.7, 41.3)
- added D11: SOD-123, Diodes_SMD:D_SOD-123, B.Cu at (223.8, 43.7)
- added D12: SOD-123, Diodes_SMD:D_SOD-123, B.Cu at (263.5, 38.9)
- added D13: SOD-123, Diodes_SMD:D_SOD-123, B.Cu at (51.6, 60.3)
- added D14: SOD-123, Diodes_SMD:D_SOD-123, B.Cu at (73.0, 60.3)
- added D15: SOD-123, Diodes_SMD:D_SOD-123, B.Cu at (92.1, 60.3)
- added D16: SOD-123, Diodes_SMD:D_SOD-123, B.Cu at (111.1, 60.3)
- added D17: SOD-123, Diodes_SMD:D_SOD-123, B.Cu at (130.2, 60.3)
- added D18: SOD-123, Diodes_SMD:D_SOD-123, B.Cu at (149.2, 60.3)
- added D19: SOD-123, Diodes_SMD:D_SOD-123, B.Cu at (168.3, 60.3)
- added D2: SOD-123, Diodes_SMD:D_SOD-123, B.Cu at (68.3, 41.3)
- added D20: SOD-123, Diodes_SMD:D_SOD-123, B.Cu at (187.3, 60.3)
- added D21: SOD-123, Diodes_SMD:D_SOD-123, B.Cu at (206.4, 60.3)
- added D22: SOD-123, Diodes_SMD:D_SOD-123, B.Cu at (225.4, 60.3)
- added D23: SOD-123, Diodes_SMD:D_SOD-123, B.Cu at (228.6, 62.7)
- added D24: SOD-123, Diodes_SMD:D_SOD-123, B.Cu at (266.7, 60.3)
- added D25: SOD-123, Diodes_SMD:D_SOD-123, B.Cu at (54.0, 79.4)
- added D26: SOD-123, Diodes_SMD:D_SOD-123, B.Cu at (77.8, 79.4)
- added D27: SOD-123, Diodes_SMD:D_SOD-123, B.Cu at (96.8, 79.4)
- added D28: SOD-123, Diodes_SMD:D_SOD-123, B.Cu at (115.9, 79.4)
- added D29: SOD-123, Diodes_SMD:D_SOD-123, B.Cu at (134.9, 79.4)
- added D3: SOD-123, Diodes_SMD:D_SOD-123, B.Cu at (87.3, 41.3)
- added D30: SOD-123, Diodes_SMD:D_SOD-123, B.Cu at (154.0, 79.4)
- added D31: SOD-123, Diodes_SMD:D_SOD-123, B.Cu at (173.0, 79.4)
- added D32: SOD-123, Diodes_SMD:D_SOD-123, B.Cu at (192.1, 79.4)
- added D33: SOD-123, Diodes_SMD:D_SOD-123, B.Cu at (211.1, 79.4)
- added D34: SOD-123, Diodes_SMD:D_SOD-123, B.Cu at (230.2, 79.4)
- added D35: SOD-123, Diodes_SMD:D_SOD-123, B.Cu at (249.2, 79.4)
- added D36: SOD-123, Diodes_SMD:D_SOD-123, B.Cu at (260.4, 84.9)
- added D37: SOD-123, Diodes_SMD:D_SOD-123, B.Cu at (49.2, 98.4)
- added D38: SOD-123, Diodes_SMD:D_SOD-123, B.Cu at (68.3, 98.4)
- added D39: SOD-123, Diodes_SMD:D_SOD-123, B.Cu at (87.3, 98.4)
- added D4: SOD-123, Diodes_SMD:D_SOD-123, B.Cu at (106.4, 41.3)
- added D40: SOD-123, Diodes_SMD:D_SOD-123, B.Cu at (106.4, 98.4)
- added D41: SOD-123, Diodes_SMD:D_SOD-123, B.Cu at (127.8, 98.4)
- added D42: SOD-123, Diodes_SMD:D_SOD-123, B.Cu at (158.8, 98.4)
- added D43: SOD-123, Diodes_SMD:D_SOD-123, B.Cu at (189.7, 98.4)
- added D44: SOD-123, Diodes_SMD:D_SOD-123, B.Cu at (211.1, 98.4)
- added D45: SOD-123, Diodes_SMD:D_SOD-123, B.Cu at (230.2, 98.4)
- added D46: SOD-123, Diodes_SMD:D_SOD-123, B.Cu at (249.2, 98.4)
- added D47: SOD-123, Diodes_SMD:D_SOD-123, B.Cu at (252.4, 100.8)
- added D5: SOD-123, Diodes_SMD:D_SOD-123, B.Cu at (125.4, 41.3)
- added D6: SOD-123, Diodes_SMD:D_SOD-123, B.Cu at (144.5, 41.3)
- added D7: SOD-123, Diodes_SMD:D_SOD-123, B.Cu at (163.5, 41.3)
- added D8: SOD-123, Diodes_SMD:D_SOD-123, B.Cu at (182.6, 41.3)
- added D9: SOD-123, Diodes_SMD:D_SOD-123, B.Cu at (201.6, 41.3)
- added MX1: MX-1U, MX_Alps_Hybrid:MXOnly-1U-Hotswap, F.Cu at (41.3, 41.3)
- added MX10: MX-1U, MX_Alps_Hybrid:MXOnly-1U-Hotswap, F.Cu at (212.7, 41.3)
- added MX11: MX-1U, MX_Alps_Hybrid:MXOnly-1U-Hotswap, F.Cu at (231.8, 41.3)
- added MX12: MX-1.5U, MX_Alps_Hybrid:MXOnly-1.5U-Hotswap, F.Cu at (255.6, 41.3)
- added MX13: MX-1.25U, MX_Alps_Hybrid:MXOnly-1.25U-Hotswap, F.Cu at (43.7, 60.3)
- added MX14: MX-1U, MX_Alps_Hybrid:MXOnly-1U-Hotswap, F.Cu at (65.1, 60.3)
- added MX15: MX-1U, MX_Alps_Hybrid:MXOnly-1U-Hotswap, F.Cu at (84.1, 60.3)
- added MX16: MX-1U, MX_Alps_Hybrid:MXOnly-1U-Hotswap, F.Cu at (103.2, 60.3)
- added MX17: MX-1U, MX_Alps_Hybrid:MXOnly-1U-Hotswap, F.Cu at (122.2, 60.3)
- added MX18: MX-1U, MX_Alps_Hybrid:MXOnly-1U-Hotswap, F.Cu at (141.3, 60.3)
- added MX19: MX-1U, MX_Alps_Hybrid:MXOnly-1U-Hotswap, F.Cu at (160.3, 60.3)
- added MX2: MX-1U, MX_Alps_Hybrid:MXOnly-1U-Hotswap, F.Cu at (60.3, 41.3)
- added MX20: MX-1U, MX_Alps_Hybrid:MXOnly-1U-Hotswap, F.Cu at (179.4, 60.3)
- added MX21: MX-1U, MX_Alps_Hybrid:MXOnly-1U-Hotswap, F.Cu at (198.4, 60.3)
- added MX22: MX-1U, MX_Alps_Hybrid:MXOnly-1U-Hotswap, F.Cu at (217.5, 60.3)
- added MX23: MX-1U, MX_Alps_Hybrid:MXOnly-1U-Hotswap, F.Cu at (236.5, 60.3)
- added MX24: MX-1.25U, MX_Alps_Hybrid:MXOnly-1.25U-Hotswap, F.Cu at (258.0, 60.3)
- added MX25: MX-1.5U, MX_Alps_Hybrid:MXOnly-1.5U-Hotswap, F.Cu at (46.0, 79.4)
- added MX26: MX-1U, MX_Alps_Hybrid:MXOnly-1U-Hotswap, F.Cu at (69.8, 79.4)
- added MX27: MX-1U, MX_Alps_Hybrid:MXOnly-1U-Hotswap, F.Cu at (88.9, 79.4)
- added MX28: MX-1U, MX_Alps_Hybrid:MXOnly-1U-Hotswap, F.Cu at (108.0, 79.4)
- added MX29: MX-1U, MX_Alps_Hybrid:MXOnly-1U-Hotswap, F.Cu at (127.0, 79.4)
- added MX3: MX-1U, MX_Alps_Hybrid:MXOnly-1U-Hotswap, F.Cu at (79.4, 41.3)
- added MX30: MX-1U, MX_Alps_Hybrid:MXOnly-1U-Hotswap, F.Cu at (146.1, 79.4)
- added MX31: MX-1U, MX_Alps_Hybrid:MXOnly-1U-Hotswap, F.Cu at (165.1, 79.4)
- added MX32: MX-1U, MX_Alps_Hybrid:MXOnly-1U-Hotswap, F.Cu at (184.2, 79.4)
- added MX33: MX-1U, MX_Alps_Hybrid:MXOnly-1U-Hotswap, F.Cu at (203.2, 79.4)
- added MX34: MX-1U, MX_Alps_Hybrid:MXOnly-1U-Hotswap, F.Cu at (222.2, 79.4)
- added MX35: MX-1U, MX_Alps_Hybrid:MXOnly-1U-Hotswap, F.Cu at (241.3, 79.4)
- added MX36: MX-1U, MX_Alps_Hybrid:MXOnly-1U-Hotswap, F.Cu at (260.4, 79.4)
- added MX37: MX-1U, MX_Alps_Hybrid:MXOnly-1U-Hotswap, F.Cu at (41.3, 98.4)
- added MX38: MX-1U, MX_Alps_Hybrid:MXOnly-1U-Hotswap, F.Cu at (60.3, 98.4)
- added MX39: MX-1U, MX_Alps_Hybrid:MXOnly-1U-Hotswap, F.Cu at (79.4, 98.4)
- added MX4: MX-1U, MX_Alps_Hybrid:MXOnly-1U-Hotswap, F.Cu at (98.4, 41.3)
- added MX40: MX-1U, MX_Alps_Hybrid:MXOnly-1U-Hotswap, F.Cu at (98.4, 98.4)
- added MX41: MX-1.25U, MX_Alps_Hybrid:MXOnly-1.25U-Hotswap, F.Cu at (119.9, 98.4)
- added MX42: MX-2U, MX_Alps_Hybrid:MXOnly-2U-Hotswap-ReversedStabilizers, F.Cu at (150.8, 98.4)
- added MX43: MX-1.25U, MX_Alps_Hybrid:MXOnly-1.25U-Hotswap, F.Cu at (181.8, 98.4)
- added MX44: MX-1U, MX_Alps_Hybrid:MXOnly-1U-Hotswap, F.Cu at (203.2, 98.4)
- added MX45: MX-1U, MX_Alps_Hybrid:MXOnly-1U-Hotswap, F.Cu at (222.2, 98.4)
- added MX46: MX-1U, MX_Alps_Hybrid:MXOnly-1U-Hotswap, F.Cu at (241.3, 98.4)
- added MX47: MX-1U, MX_Alps_Hybrid:MXOnly-1U-Hotswap, F.Cu at (260.4, 98.4)
- added MX5: MX-1U, MX_Alps_Hybrid:MXOnly-1U-Hotswap, F.Cu at (117.5, 41.3)
- added MX6: MX-1U, MX_Alps_Hybrid:MXOnly-1U-Hotswap, F.Cu at (136.5, 41.3)
- added MX7: MX-1U, MX_Alps_Hybrid:MXOnly-1U-Hotswap, F.Cu at (155.6, 41.3)
- added MX8: MX-1U, MX_Alps_Hybrid:MXOnly-1U-Hotswap, F.Cu at (174.6, 41.3)
- added MX9: MX-1U, MX_Alps_Hybrid:MXOnly-1U-Hotswap, F.Cu at (193.7, 41.3)
- added R6: 5.1k, Resistors_SMD:R_0603, B.Cu at (242.1, 42.1)
- added U2: PRTR5V0U2X, locallib:SOT143B, B.Cu at (246.6, 42.0)
- C1, C2, C3, C4, C5, C6, CR1, CR2, CR3, CR4, CR5, CR6, CR7, CR8: footprint Capacitors_SMD:C_0805_HandSoldering -> Capacitors_SMD:C_0603
- F1: footprint Fuse_Holders_and_Fuses:Fuse_SMD1206_HandSoldering -> Fuse_Holders_and_Fuses:Fuse_SMD1206_Reflow
- R1, R2, R3, R5: footprint Resistors_SMD:R_0805_HandSoldering -> Resistors_SMD:R_0603
- R4: value 1.5k -> 5.1k; footprint Resistors_SMD:R_0805_HandSoldering -> Resistors_SMD:R_0603
- SW1: footprint Molex-0548190589:PushButton_6x6mm_TH -> Molex-0548190589:SKQG-1155865
- U1: footprint Housings_QFP:TQFP-32_7x7mm_Pitch0.8mm -> Housings_DFN_QFN:QFN-32-1EP_5x5mm_Pitch0.5mm
- USB1: value Molex-0548190589 -> HRO-TYPE-C-31-M-12; footprint Molex-0548190589:Molex-0548190589 -> Type-C:HRO-TYPE-C-31-M-12-Assembly
- Y1: footprint Crystals:Crystal_SMD_3225-4pin_3.2x2.5mm_HandSoldering -> Crystals:Crystal_SMD_3225-4pin_3.2x2.5mm
- moved CR5 259.5 mm to (50.8, 83.3), turned to 180 degrees
- moved RGB5 253.1 mm to (50.8, 87.3)
- moved CR4 230.8 mm to (50.8, 45.2), turned to 180 degrees
- moved RGB4 223.9 mm to (50.8, 49.2)
- moved USB1 180.9 mm to (246.0, 30.2), turned to 0 degrees
- moved R3 180.2 mm to (246.7, 54.5), turned to 180 degrees
- moved RGB6 179.0 mm to (117.5, 87.3)
- moved R2 177.4 mm to (246.7, 56.7), turned to 0 degrees
- moved CR6 172.9 mm to (117.5, 83.3), turned to 180 degrees
- moved F1 172.4 mm to (234.8, 46.4), turned to 0 degrees
- moved SW1 154.9 mm to (231.8, 87.3), turned to 180 degrees
- moved C1 141.0 mm to (255.2, 63.8), turned to 0 degrees
- moved R4 137.1 mm to (253.2, 36.5), turned to 90 degrees
- moved C2 136.0 mm to (255.2, 66.0)
- moved Y1 134.2 mm to (250.9, 64.9), turned to 270 degrees
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Connections:
- R2 pad 1: /D_P -> D-
- R2 pad 2: DP -> Net-(R2-Pad2)
- R3 pad 1: /D_N -> Net-(R3-Pad1)
- R3 pad 2: DM -> D+
- R4 pad 1: Net-(Q1-Pad1) -> Net-(R4-Pad1)
- R4 pad 2: Net-(R4-Pad2) -> GND
- U1 pad 10: ROW1 -> Net-(U1-Pad10)
- U1 pad 11: ROW4 -> Net-(U1-Pad11)
- U1 pad 12: ROW3 -> Net-(U1-Pad12)
- U1 pad 14: ROW2 -> Net-(U1-Pad14)
- U1 pad 15: ROW5 -> Net-(U1-Pad15)
- U1 pad 16: ROW6 -> Net-(U1-Pad16)
- U1 pad 17: COL4 -> Net-(U1-Pad17)
- U1 pad 18: COL5 -> Net-(U1-Pad18)
- U1 pad 19: COL6 -> Net-(U1-Pad19)
- U1 pad 20: COL7 -> Net-(U1-Pad20)
- U1 pad 21: Net-(R4-Pad2) -> Net-(U1-Pad21)
- U1 pad 22: RGBLED -> Net-(U1-Pad22)
- U1 pad 23: COL3 -> Net-(U1-Pad23)
- U1 pad 25: ROW8 -> Net-(U1-Pad25)
- U1 pad 26: ROW9 -> Net-(U1-Pad26)
- U1 pad 29: /D_P -> D+
- U1 pad 30: /D_N -> D-
- U1 pad 5: COL1 -> Net-(U1-Pad5)
- U1 pad 6: COL0 -> Net-(U1-Pad6)
- U1 pad 7: ROW7 -> Net-(U1-Pad7)
- U1 pad 8: COL2 -> Net-(U1-Pad8)
- U1 pad 9: ROW0 -> Net-(U1-Pad9)
- USB1 pad 2: Net-(USB1-Pad2) -> VCC
- USB1 pad 3: DP -> Net-(USB1-Pad3)
- USB1 pad 4: DM -> Net-(R6-Pad1)
- USB1 pad 5: VCC -> Net-(R2-Pad2)
Routing:
- net LEDGND: track 1378.1 -> 0.00 mm, vias 20 -> 0
- net +5V: track 1924.8 -> 548.0 mm, vias 20 -> 6
- net ROW8: track 335.8 -> 0.00 mm, vias 4 -> 0
- net COL6: track 344.1 -> 48.6 mm
- net ROW9: track 284.6 -> 0.00 mm, vias 4 -> 0
- net ROW5: track 276.3 -> 0.00 mm, vias 2 -> 0
- net ROW6: track 261.7 -> 0.00 mm, vias 2 -> 0
- net COL5: track 327.2 -> 71.8 mm, vias 3 -> 4
- net ROW4: track 250.9 -> 0.00 mm, vias 2 -> 0
- net ROW7: track 243.5 -> 0.00 mm, vias 2 -> 0
- net COL7: track 309.9 -> 70.7 mm, vias 3 -> 4
- net GND: track 857.7 -> 647.3 mm, vias 28 -> 22
- net COL4: track 249.6 -> 72.7 mm, vias 3 -> 4
- net /D_P: track 167.0 -> 0.00 mm, vias 2 -> 0
- net /D_N: track 166.4 -> 0.00 mm, vias 2 -> 0
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- removed copper zone on B.Cu, net GND
- removed copper zone on F.Cu, net GND
Other:
- board size 285 x 94.6 mm -> 238.1 x 76.2 mm
- board text removed: "60% keyboard PCB Designed by ai03 60% outline by amtra5"
- board text removed: "An endless journey into the unknown."
- board text removed: "Rev. 2.0"
- board text removed: "VOYAGER"
- board text removed: "www.ai03.me"
