File: Mir.kicad_pcb (KiCad board)
At the start: 2 copper layers, 238.1 x 76.2 mm, 128 parts, among them SW1 SW_PUSH, U1 ATMEGA32U2-AU, U2 PRTR5V0U2X, Y1 16MHz

Commit message: Finish routing
Connections:
- U1 pad 10: Net-(U1-Pad10) -> ROW3
- U1 pad 11: Net-(U1-Pad11) -> COL11
- U1 pad 12: Net-(U1-Pad12) -> COL10
- U1 pad 14: Net-(U1-Pad14) -> COL9
- U1 pad 15: Net-(U1-Pad15) -> COL8
- U1 pad 16: Net-(U1-Pad16) -> COL7
- U1 pad 17: Net-(U1-Pad17) -> COL6
- U1 pad 18: Net-(U1-Pad18) -> COL5
- U1 pad 19: Net-(U1-Pad19) -> COL4
- U1 pad 20: Net-(U1-Pad20) -> COL3
- U1 pad 21: Net-(U1-Pad21) -> COL2
- U1 pad 25: Net-(U1-Pad25) -> COL1
- U1 pad 26: Net-(U1-Pad26) -> COL0
- U1 pad 7: Net-(U1-Pad7) -> ROW0
- U1 pad 8: Net-(U1-Pad8) -> ROW1
- U1 pad 9: Net-(U1-Pad9) -> ROW2
Routing:
- net COL0: track 69.8 -> 278.9 mm
- net COL1: track 73.7 -> 257.6 mm
- net COL2: track 73.7 -> 236.9 mm
- net COL3: track 73.7 -> 217.6 mm
- net COL4: track 72.7 -> 197.3 mm
- net COL5: track 71.8 -> 177.1 mm
- net COL6: track 48.6 -> 134.7 mm
- net COL7: track 70.7 -> 138.2 mm
- net ROW0: track 227.5 -> 278.4 mm, vias 2 -> 4
- net COL8: track 69.8 -> 119.0 mm
- net ROW3: track 211.2 -> 247.8 mm, vias 0 -> 2
- net COL9: track 69.8 -> 100.6 mm
- net ROW1: track 237.2 -> 266.2 mm
- net ROW2: track 216.0 -> 232.2 mm, vias 0 -> 2
- net COL10: track 69.8 -> 83.6 mm
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- added copper zone on B.Cu, net GND
Other:
- net class POWER: trace_width 0.381 -> 0.635

Commit message: Decorations
Parts:
- added G***: LOGO, locallib:ai-ring-6mm-FancyAss, B.Cu at (265.1, 103.2)
- added G***: LOGO, locallib:ai-ring-6mm-FancyAss-Mask, B.Cu at (265.1, 103.2)
- added G***: LOGO, locallib:Keyhive-Silk, F.Cu at (150.8, 69.8)
- moved D24 0.79 mm to (265.9, 60.3)
Connections:
- U1 pad 23: Net-(U1-Pad23) -> RGBLED
Routing:
- net RGBLED: track 2.39 -> 24.2 mm, vias 1 -> 2
- net GND: track 650.4 -> 656.4 mm
- net +5V: track 543.4 -> 538.0 mm
- net ROW1: track 266.2 -> 264.6 mm
Other:
- board text added: "Distributed by Keyhive | 20181128 | Credits to 40percent.club's Gnap"
- board text added: "UT47.2"
- board text added: "UT47.2 PCB by ai03 Rev 1.0"

Commit message: Error check
Routing:
- net +5V: track 538.0 -> 538.5 mm
Changed lines of the file:
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@@
     (tags SOD-123)
     (attr smd)
-    (fp_text reference D22 (at 0 2 90) (layer B.SilkS)
+    (fp_text reference D22 (at -3.96875 0 90) (layer B.SilkS)
       (effects (font (size 1 1) (thickness 0.15)) (justify mirror))
     )
@@
   (segment (start 233.045 50.292) (end 237.363 50.292) (width 0.381) (layer B.Cu) (net 2))
   (segment (start 233.045 50.292) (end 232.664 49.911) (width 0.381) (layer B.Cu) (net 2))
-  (segment (start 238.76 66.167) (end 241.3 66.167) (width 0.635) (layer F.Cu) (net 2))
-  (segment (start 242.951 64.516) (end 242.951 61.722) (width 0.635) (layer F.Cu) (net 2))
-  (segment (start 241.3 66.167) (end 242.951 64.516) (width 0.635) (layer F.Cu) (net 2))
-  (segment (start 236.728 64.135) (end 234.823 64.135) (width 0.635) (layer F.Cu) (net 2))
-  (segment (start 236.728 64.135) (end 238.76 66.167) (width 0.635) (layer F.Cu) (net 2))
   (segment (start 234.569 63.881) (end 234.823 64.135) (width 0.635) (layer F.Cu) (net 2))
   (segment (start 234.569 63.5) (end 234.569 63.881) (width 0.635) (layer F.Cu) (net 2))
@@
   (segment (start 234.823 71.12) (end 233.807 70.104) (width 0.635) (layer F.Cu) (net 2))
   (segment (start 240.03 71.12) (end 234.823 71.12) (width 0.635) (layer F.Cu) (net 2))
+  (segment (start 242.951 64.516) (end 242.951 61.722) (width 0.635) (layer F.Cu) (net 2))
+  (segment (start 241.3 66.167) (end 242.951 64.516) (width 0.635) (layer F.Cu) (net 2))
+  (segment (start 239.649 66.167) (end 241.3 66.167) (width 0.635) (layer F.Cu) (net 2))
+  (segment (start 237.617 64.135) (end 239.649 66.167) (width 0.635) (layer F.Cu) (net 2))
+  (segment (start 234.823 64.135) (end 237.617 64.135) (width 0.635) (layer F.Cu) (net 2))
   (segment (start 254.42475 65.9765) (end 253.9365 65.9765) (width 0.25) (layer B.Cu) (net 3))
   (segment (start 253.9365 65.9765) (end 252.73 67.183) (width 0.25) (layer B.Cu) (net 3))
@@
   (segment (start 233.934 47.993) (end 236.601 47.993) (width 0.381) (layer B.Cu) (net 5))
   (segment (start 236.601 47.993) (end 237.122 47.993) (width 0.381) (layer B.Cu) (net 5))
-  (segment (start 236.855 65.913) (end 238.125 67.183) (width 0.635) (layer F.Cu) (net 5))
-  (segment (start 234.696 65.913) (end 236.855 65.913) (width 0.635) (layer F.Cu) (net 5))
-  (segment (start 241.3 67.183) (end 241.808 67.183) (width 0.635) (layer F.Cu) (net 5))
-  (segment (start 238.125 67.183) (end 241.3 67.183) (width 0.635) (layer F.Cu) (net 5))
-  (segment (start 241.808 67.183) (end 243.967 65.024) (width 0.635) (layer F.Cu) (net 5))
   (segment (start 243.967 62.103) (end 244.475 61.595) (width 0.635) (layer F.Cu) (net 5))
   (segment (start 243.967 65.024) (end 243.967 62.103) (width 0.635) (layer F.Cu) (net 5))
   (segment (start 243.967 65.659) (end 243.967 65.024) (width 0.635) (layer F.Cu) (net 5))
   (segment (start 244.475 66.167) (end 243.967 65.659) (width 0.635) (layer F.Cu) (net 5))
+  (segment (start 241.808 67.183) (end 243.967 65.024) (width 0.635) (layer F.Cu) (net 5))
+  (segment (start 239.141 67.183) (end 241.808 67.183) (width 0.635) (layer F.Cu) (net 5))
+  (segment (start 237.236 65.278) (end 239.141 67.183) (width 0.635) (layer F.Cu) (net 5))
+  (segment (start 235.331 65.278) (end 237.236 65.278) (width 0.635) (layer F.Cu) (net 5))
+  (segment (start 234.696 65.913) (end 235.331 65.278) (width 0.635) (layer F.Cu) (net 5))
   (segment (start 223.8375 45.30625) (end 222.34425 45.30625) (width 0.25) (layer B.Cu) (net 6))
   (segment (start 220.6625 43.6245) (end 220.6625 42.925) (width 0.25) (layer B.Cu) (net 6))
