File: UT47.2.kicad_pcb (KiCad board)
At the start: 2 copper layers, 238.1 x 76.2 mm, 131 parts, among them SW1 SW_PUSH, U1 ATMEGA32U2-AU, U2 PRTR5V0U2X, Y1 16MHz

Commit message: Fix position files
Parts:
- RGB1, RGB2, RGB3, RGB4, RGB5, RGB6, RGB7, RGB8: value WS2812B -> VAL**
