File: UT47.2.kicad_pcb (KiCad board)
At the start: 2 copper layers, 238.1 x 76.2 mm, 131 parts, among them SW1 SW_PUSH, U1 ATMEGA32U2-AU, U2 PRTR5V0U2X, Y1 16MHz

Commit message: Finally get KiCad to print properly
Other:
- board text added: "RGB1"
- board text added: "RGB2"
- board text added: "RGB3"
- board text added: "RGB4"
- board text added: "RGB5"
- board text added: "RGB6"
- board text added: "RGB7"
- board text added: "RGB8"
