File: UT47.2.kicad_pcb (KiCad board)
At the start: 2 copper layers, 238.1 x 76.2 mm, 131 parts, among them SW1 SW_PUSH, U1 ATMEGA32U2-AU, U2 PRTR5V0U2X, Y1 16MHz

Commit message: Update with drill holes
Parts:
- added REF**: MountingHole_2.2mm_M2_Pad_Via, Mounting_Holes:MountingHole_2.2mm_M2_Pad_Via, F.Cu at (150.8, 69.8)
- added REF**: MountingHole_2.2mm_M2_Pad_Via, Mounting_Holes:MountingHole_2.2mm_M2_Pad_Via, F.Cu at (41.3, 88.9)
- added REF**: MountingHole_2.2mm_M2_Pad_Via, Mounting_Holes:MountingHole_2.2mm_M2_Pad_Via, F.Cu at (41.3, 50.8)
- added REF**: MountingHole_2.2mm_M2_Pad_Via, Mounting_Holes:MountingHole_2.2mm_M2_Pad_Via, F.Cu at (260.4, 50.8)
- added REF**: MountingHole_2.2mm_M2_Pad_Via, Mounting_Holes:MountingHole_2.2mm_M2_Pad_Via, F.Cu at (260.4, 88.9)
- moved D36 5.78 mm to (265.9, 83.3)
Routing:
- net ROW2: track 232.2 -> 237.1 mm
- net Net-(D36-Pad2): track 11.9 -> 8.04 mm
- net COL5: track 177.1 -> 178.9 mm
- net COL4: track 197.3 -> 199.1 mm
- net COL2: track 236.9 -> 238.6 mm
- net COL3: track 217.6 -> 219.4 mm
- net COL1: track 257.9 -> 259.7 mm
- net COL0: track 278.9 -> 280.7 mm
Other:
- net class POWER: trace_width 0.635 -> 0.381
- board text added: "kb.ai03.me"
- board text removed: "UT47.2 PCB by ai03 Rev 1.0"
