File: Case Files/Bottom/UT47.2-Bottom.kicad_pcb (KiCad board)
At the start: 2 copper layers, 254.1 x 92.2 mm, 2 parts, among them J1 Outline

Commit message: New case data
Parts:
- added G***: LOGO, locallib:hex, F.Cu at (146.8, 68.3)
- G***: moved to B.Cu
- moved G*** 227.0 mm to (33.3, 100.5), turned to 180 degrees
